File: IO_Experiments Board.sch (EAGLE design)
At the start: 191 parts, among them IC1 ULN2803, IC10 ULN2803, IC11 NX1117CE33Z, IC13 L298, IC2 4511N, IC3 PCF8563P, IC4 MCP23017SP, IC5 MAX7219CNG, IC6 74125N, IC7 AT24CP, IC8 MCP23017SP, IC9 MCP23017SP, K1 G2RA, K2 G2RA, K3 G2RA, K4 G2RA, K5 G2RA, K6 G2RA, K7 G2RA, K8 G2RA, Q1 32.768 kHz, SW1 EC12E_SW, T1 BC547, T2 BC547, T3 BC547, T4 BC547, U2 JOYSTICK, X2 POWERSUPPLY_DC21MMX

Commit message: added signal names on connectors on the board , layer 51
Connections:
- net N$116 renamed REL1
- net N$120 renamed REL2
- net N$121 renamed REL3
- net N$122 renamed 2A0
- net N$123 renamed 2A1
- net N$124 renamed 2A2
- net N$125 renamed 2A3
- net N$126 renamed 2A4
- net N$127 renamed 2A5
- net N$128 renamed 2A6
- net N$129 renamed 2A7
- net N$130 renamed 2B0
- net N$131 renamed 2B1
- net N$132 renamed 2B2
- net N$133 renamed 2B3
- net N$134 renamed 2B4
- net N$135 renamed 2B5
- net N$136 renamed 2B6
- net N$137 renamed 2B7
- net N$141 renamed 3A0
- net N$142 renamed 3A1
- net N$143 renamed 3A2
- net N$144 renamed 3A3
- net N$145 renamed 3A4
- net N$146 renamed 3A5
- net N$147 renamed 3A6
- net N$148 renamed 3A7
- net N$149 renamed 3B0
- net N$150 renamed 3B1
- net N$151 renamed 3B2
- net N$152 renamed 3B3
- net N$153 renamed 3B4
- net N$154 renamed 3B5
- net N$155 renamed 3B6
- net N$156 renamed 3B7
- net N$160 renamed REL4
- net N$161 renamed REL5
- net N$162 renamed REL6
- net N$163 renamed REL7
- net N$164 renamed REL8
- net N$25 renamed CONTRAST
- net N$27 renamed LCD_E
- net N$35 renamed LCD_RW
- net N$36 renamed LCD_RS
- net N$37 renamed LCD_D0
- net N$38 renamed LCD_D1
- net N$39 renamed LCD_D2
- net N$40 renamed LCD_D3
- net N$41 renamed LCD_D4
- net N$42 renamed LCD_D5
- net N$43 renamed LCD_D6
- net N$44 renamed LCD_D7
- net N$60 renamed IA
- net N$61 renamed IB
- net N$62 renamed IC
- net N$63 renamed ID
- net N$64 renamed D1
- net N$65 renamed D2
- net N$66 renamed D3
- net N$67 renamed D4
- net N$68 renamed 1A0
- net N$69 renamed 1A1
- net N$70 renamed 1A2
- net N$71 renamed 1A3
- net N$72 renamed 1A4
- net N$75 renamed 1A5
- net N$76 renamed 1A6
- net N$77 renamed 1A7
- net N$78 renamed 1B0
- net N$79 renamed 1B1
- net N$80 renamed 1B2
- net N$81 renamed 1B3
- net N$82 renamed 1B4
- net N$83 renamed 1B5
- net N$84 renamed 1B6
- net N$85 renamed 1B7
